File: esp_sonar.kicad_sch (KiCad schematic)
At the start: 16 parts, among them J1 Conn_01x04_Male, Q1 2N4401, Q2 BS250, Q3 2N7000

Commit message: Replaced high-side mosfet with resistor to prevent shoot-through
Parts:
- removed Q2: BS250, Package_TO_SOT_THT:TO-92_Inline, symbol Transistor_FET:BS250
- R5: value 100k -> 100; footprint Resistor_THT:R_Axial_DIN0207_L6.3mm_D2.5mm_P2.54mm_Vertical -> Resistor_THT:R_Axial_DIN0207_L6.3mm_D2.5mm_P5.08mm_Vertical
Connections:
- net +5V: now also R5.1
- net GND: no longer R5.2
- net TX: no longer R5.1
- net at LS1.1, Q3.3 (D): now also R5.2
Changed lines of the file:
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@@
   (junction (at 93.98 66.04) (diameter 0) (color 0 0 0 0)
   )
-  (junction (at 107.95 64.77) (diameter 0) (color 0 0 0 0)
-  )
   (junction (at 119.38 114.3) (diameter 0) (color 0 0 0 0)
   )
@@
   (junction (at 107.95 114.3) (diameter 0) (color 0 0 0 0)
   )
-  (wire (pts (xy 107.95 64.77) (xy 111.76 64.77))
-    (stroke (width 0) (type default) (color 0 0 0 0))
-  )
   (wire (pts (xy 115.57 111.76) (xy 115.57 114.3))
     (stroke (width 0) (type default) (color 0 0 0 0))
@@
     (stroke (width 0) (type default) (color 0 0 0 0))
   )
-  (wire (pts (xy 107.95 64.77) (xy 107.95 71.12))
-    (stroke (width 0) (type default) (color 0 0 0 0))
-  )
   (wire (pts (xy 107.95 111.76) (xy 107.95 114.3))
     (stroke (width 0) (type default) (color 0 0 0 0))
@@
     (stroke (width 0) (type default) (color 0 0 0 0))
   )
-  (wire (pts (xy 101.6 64.77) (xy 107.95 64.77))
+  (wire (pts (xy 101.6 64.77) (xy 111.76 64.77))
     (stroke (width 0) (type default) (color 0 0 0 0))
   )
@@
     (stroke (width 0) (type default) (color 0 0 0 0))
   )
-  (wire (pts (xy 93.98 63.5) (xy 93.98 66.04))
+  (wire (pts (xy 93.98 60.96) (xy 93.98 66.04))
     (stroke (width 0) (type default) (color 0 0 0 0))
   )
@@
     (pin "2")
   )
-  (symbol (lib_id "power:GND") (at 107.95 78.74 0) (unit 1)
-    (in_bom yes) (on_board yes) (fields_autoplaced)
-    (property "Reference" "#PWR08" (id 0) (at 107.95 85.09 0)
-      (effects (font (size 1.27 1.27)) hide)
-    )
-    (property "Value" "GND" (id 1) (at 107.95 83.82 0))
-    (property "Footprint" "" (id 2) (at 107.95 78.74 0)
-      (effects (font (size 1.27 1.27)) hide)
-    )
-    (property "Datasheet" "" (id 3) (at 107.95 78.74 0)
-      (effects (font (size 1.27 1.27)) hide)
-    )
-    (pin "1")
-  )
-  (symbol (lib_id "Device:R_US") (at 107.95 74.93 0) (unit 1)
-    (in_bom yes) (on_board yes) (fields_autoplaced)
-    (property "Reference" "R5" (id 0) (at 110.49 73.6599 0)
-      (effects (font (size 1.27 1.27)) (justify left))
-    )
-    (property "Value" "100k" (id 1) (at 110.49 76.1999 0)
-      (effects (font (size 1.27 1.27)) (justify left))
-    )
-    (property "Footprint" "Resistor_THT:R_Axial_DIN0207_L6.3mm_D2.5mm_P2.54mm_Vertical" (id 2) (at 108.966 75.184 90)
-      (effects (font (size 1.27 1.27)) hide)
-    )
-    (property "Datasheet" "~" (id 3) (at 107.95 74.93 0)
-      (effects (font (size 1.27 1.27)) hide)
-    )
-    (pin "1")
-    (pin "2")
-  )
   (symbol (lib_id "Device:R_US") (at 119.38 119.38 0) (unit 1)
     (in_bom yes) (on_board yes) (fields_autoplaced)
@@
     )
     (pin "1")
+  )
+  (symbol (lib_id "Device:R_US") (at 93.98 57.15 0) (unit 1)
+    (in_bom yes) (on_board yes) (fields_autoplaced)
+    (property "Reference" "R5" (id 0) (at 96.52 55.8799 0)
+      (effects (font (size 1.27 1.27)) (justify left))
+    )
+    (property "Value" "100" (id 1) (at 96.52 58.4199 0)
+      (effects (font (size 1.27 1.27)) (justify left))
+    )
+    (property "Footprint" "Resistor_THT:R_Axial_DIN0207_L6.3mm_D2.5mm_P5.08mm_Vertical" (id 2) (at 94.996 57.404 90)
+      (effects (font (size 1.27 1.27)) hide)
+    )
+    (property "Datasheet" "~" (id 3) (at 93.98 57.15 0)
+      (effects (font (size 1.27 1.27)) hide)
+    )
+    (pin "1")
+    (pin "2")
   )
   (symbol (lib_id "power:+5V") (at 119.38 105.41 0) (unit 1)
@@
     (pin "2")
   )
-  (symbol (lib_id "Transistor_FET:BS250") (at 96.52 58.42 180) (unit 1)
-    (in_bom yes) (on_board yes) (fields_autoplaced)
-    (property "Reference" "Q2" (id 0) (at 90.17 57.1499 0)
-      (effects (font (size 1.27 1.27)) (justify left))
-    )
-    (property "Value" "BS250" (id 1) (at 90.17 59.6899 0)
-      (effects (font (size 1.27 1.27)) (justify left))
-    )
-    (property "Footprint" "Package_TO_SOT_THT:TO-92_Inline" (id 2) (at 91.44 56.515 0)
-      (effects (font (size 1.27 1.27) italic) (justify left) hide)
-    )
-    (property "Datasheet" "http://www.vishay.com/docs/70209/70209.pdf" (id 3) (at 96.52 58.42 0)
-      (effects (font (size 1.27 1.27)) (justify left) hide)
-    )
-    (pin "1")
-    (pin "2")
-    (pin "3")
-  )
   (symbol (lib_id "kamocat:2N4401") (at 69.85 121.92 0) (unit 1)
     (in_bom yes) (on_board yes) (fields_autoplaced)
@@
       (reference "#PWR07") (unit 1) (value "GND") (footprint "")
     )
-    (path "/46c62521-3389-4214-8f35-9a2436fc56ac"
-      (reference "#PWR08") (unit 1) (value "GND") (footprint "")
-    )
     (path "/2c59491a-3564-4661-a789-5350cc5b0011"
       (reference "#PWR0101") (unit 1) (value "GND") (footprint "")
@@
       (reference "Q1") (unit 1) (value "2N4401") (footprint "Package_TO_SOT_THT:TO-92_Inline_Wide")
     )
-    (path "/fe678902-5fe5-404f-8c39-57bf9918a117"
-      (reference "Q2") (unit 1) (value "BS250") (footprint "Package_TO_SOT_THT:TO-92_Inline")
-    )
     (path "/2638ab6f-7c7b-4642-ad60-8e9d6c13acc9"
       (reference "Q3") (unit 1) (value "2N7000") (footprint "Package_TO_SOT_THT:TO-92_Inline")
@@
       (reference "R4") (unit 1) (value "100k") (footprint "Resistor_THT:R_Axial_DIN0207_L6.3mm_D2.5mm_P10.16mm_Horizontal")
     )
-    (path "/5b0b81f7-99d8-4b9e-8bf6-3f4b56a1f4f0"
-      (reference "R5") (unit 1) (value "100k") (footprint "Resistor_THT:R_Axial_DIN0207_L6.3mm_D2.5mm_P2.54mm_Vertical")
-    )
-  )
+    (path "/9660c60c-1158-471c-ba82-ec520035cdb6"
+      (reference "R5") (unit 1) (value "100") (footprint "Resistor_THT:R_Axial_DIN0207_L6.3mm_D2.5mm_P5.08mm_Vertical")
+    )
+  )
